File: Spring 2023/Electrical/Eagle Files/strato_cats/schematic.brd (EAGLE design)
At the start: 124.1 x 119.4 mm, 21 parts

Commit message: finished board
Parts:
- removed J4, J9: (no value), SparkFun-Connectors:1X06_NO_SILK
- removed JP2: (no value), microbuilder:1X07_ROUND_70
- removed JP4: (no value), adafruit:1X08-BIG
- removed U$47, U$74: (no value), buzzard_labels_2:GND4
- removed U$62: (no value), buzzard_labels_2:MISO13
- removed U$63: (no value), buzzard_labels_2:MOSI14
- removed U$64: (no value), buzzard_labels_2:SCLK15
- removed U$65: (no value), buzzard_labels_2:#CS16
- removed U$66: (no value), buzzard_labels_2:1V8#5V57
- removed U$67: (no value), buzzard_labels_2:VIN5
- removed U$68: (no value), buzzard_labels_2:NC17
- removed U$69: (no value), buzzard_labels_2:AD012
- removed U$89: (no value), buzzard_labels:CL4
- removed U$90: (no value), buzzard_labels:DA2
- added 9DOF_1, 9DOF_2: (no value), SparkFun-Connectors:1X06_NO_SILK
- added BATT: (no value), SparkFun-Connectors:1X02
- added BME: (no value), microbuilder:1X07_ROUND_70
- added EXTRA_IO: (no value), SparkFun-Connectors:1X06
- added GEIGER: (no value), SparkFun-Connectors:1X04
- added SD_R: (no value), adafruit:1X08-BIG
- renumbered B1 to ARDUINO, J2 to GRAV, JP3 to GUVA
Connections:
- removed net !CS!_VIN: ARDUINO.7, J4.6
- removed net +3V3: JP4.2
- removed net 5V*3: ARDUINO.5V, ARDUINO.5V@1, ARDUINO.5V@2, GRAV.1, GUVA.1, J4.2, J9.6, JP2.1, JP4.1
- removed net AD0/SDO_VIN: J4.5
- removed net AUX_CL_VIN: J9.5
- removed net AUX_DA_VIN: J9.4
- removed net CD: JP4.8
- removed net DI: ARDUINO.51, JP4.6
- removed net DO: ARDUINO.50, JP4.5
- removed net FSYNC_VIN: J9.3
- removed net INT_VIN: J9.2
- removed net N$2: JP2.2
- removed net SDA/SDI_VIN: ARDUINO.20, GRAV.4, J4.3, JP2.6
- removed net SDO/ADR: JP2.5
- new net 3V: 9DOF_1.2
- new net 5V: ARDUINO.5V, ARDUINO.5V@1, ARDUINO.5V@2, BATT.1, BME.1, EXTRA_IO.5, GEIGER.3, GRAV.1, GUVA.1, SD_R.1
- new net D4: ARDUINO.4, EXTRA_IO.1
- new net D5: ARDUINO.5, EXTRA_IO.2
- new net DS: ARDUINO.3, GEIGER.2
- new net NS: ARDUINO.2, GEIGER.1
- new net SDA: 9DOF_1.3, ARDUINO.SDA, BME.6, EXTRA_IO.4, GRAV.4
- new net SDI: ARDUINO.51, SD_R.6
- new net SDO: ARDUINO.50, SD_R.5
- net CLK: now also SD_R.4; no longer JP4.4
- net CS: now also SD_R.7; no longer JP2.7, JP4.7
- net GND: now also 9DOF_1.1, 9DOF_2.1, ARDUINO.GND@1, ARDUINO.GND@2, BATT.2, BME.3, EXTRA_IO.6, GEIGER.4, SD_R.3; no longer J4.1, J9.1, JP2.3, JP4.3
- net SCL: now also 9DOF_1.4, ARDUINO.SCL, BME.4, EXTRA_IO.3; no longer ARDUINO.21, J4.4, JP2.4
Routing:
- net 5V: track 0.00 -> 241.3 mm, vias 0 -> 1
- net SCL: track 0.00 -> 153.9 mm
- net SDA: track 0.00 -> 136.8 mm
- net CS: track 0.00 -> 58.7 mm
- net N$1: track 0.00 -> 53.3 mm
- net D4: track 0.00 -> 49.8 mm
- net D5: track 0.00 -> 47.3 mm
- net SDI: track 0.00 -> 44.1 mm, vias 0 -> 1
- net NS: track 0.00 -> 29.2 mm
- net DS: track 0.00 -> 22.2 mm
- net SDO: track 0.00 -> 15.7 mm
- net CLK: track 0.00 -> 15.2 mm
- added copper zone on layer 1, net GND
- added copper zone on layer 16, net GND
Other:
- board size 124.1 x 119.4 mm -> 111.8 x 78.7 mm
- board text added: "3v"
- board text added: "5V ready Micro-SD"
- board text added: "5v"
- board text added: "Breakout board+"
- board text added: "CD"
- board text added: "CLK"
- board text added: "CS"
- board text added: "DI"
- board text added: "DO"
- board text added: "adafruit.com"
- board text removed: "Owen Lyke"

Commit message: final board !
Routing:
- net NS: track 29.2 -> 28.2 mm
Other:
- board text added: "UA ASCEND Spring 2023"
Changed lines of the file:
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@@
 <wire x1="-6.35" y1="3.81" x2="105.41" y2="3.81" width="0.1524" layer="20"/>
 <wire x1="105.41" y1="3.81" x2="105.41" y2="82.55" width="0.1524" layer="20"/>
+<text x="-2.667" y="9.017" size="1.778" layer="21" rot="R90">UA ASCEND Spring 2023</text>
+<text x="74.676" y="5.207" size="1.778" layer="21">UA ASCEND Spring 2023</text>
 </plain>
 <attributes>
@@
 </class>
 </classes>
-<designrules name="default *">
-<description language="de">&lt;b&gt;EAGLE Design Rules&lt;/b&gt;
+<designrules name="DRC">
+<description language="en">&lt;b&gt;OSH Park Design Rules&lt;/b&gt;
 &lt;p&gt;
-Die Standard-Design-Rules sind so gewählt, dass sie für
-die meisten Anwendungen passen. Sollte ihre Platine
-besondere Anforderungen haben, treffen Sie die erforderlichen
-Einstellungen hier und speichern die Design Rules unter
-einem neuen Namen ab.</description>
-<description language="en">&lt;b&gt;EAGLE Design Rules&lt;/b&gt;
+Please make sure your boards conform to these design rules.
+&lt;/p&gt;
 &lt;p&gt;
-The default Design Rules have been set to cover
-a wide range of applications. Your particular design
-may have different requirements, so please make the
-necessary adjustments and save your customized
-design rules under a new name.</description>
+Note, that not all DRC settings must be set by the manufacturer. Several can be adjusted for the design, including those listed on our docs page here.
+&lt;a href=&quot;http://docs.oshpark.com/design-tools/eagle/design-rules-files/&quot;&gt;Adjustable Settings&lt;/a&gt;
+&lt;/p&gt;</description>
 <param name="layerSetup" value="(1*16)"/>
-<param name="mtCopper" value="0.035mm 0.035mm 0.035mm 0.035mm 0.035mm 0.035mm 0.035mm 0.035mm 0.035mm 0.035mm 0.035mm 0.035mm 0.035mm 0.035mm 0.035mm 0.035mm"/>
-<param name="mtIsolate" value="1.5mm 0.15mm 0.2mm 0.15mm 0.2mm 0.15mm 0.2mm 0.15mm 0.2mm 0.15mm 0.2mm 0.15mm 0.2mm 0.15mm 0.2mm"/>
-<param name="mdWireWire" value="15mil"/>
-<param name="mdWirePad" value="15mil"/>
-<param name="mdWireVia" value="15mil"/>
-<param name="mdPadPad" value="15mil"/>
-<param name="mdPadVia" value="15mil"/>
-<param name="mdViaVia" value="15mil"/>
-<param name="mdSmdPad" value="15mil"/>
-<param name="mdSmdVia" value="15mil"/>
-<param name="mdSmdSmd" value="15mil"/>
-<param name="mdViaViaSameLayer" value="6mil"/>
+<param name="mtCopper" value="0.035559375mm 0.0356mm 0.0356mm 0.0356mm 0.0356mm 0.0356mm 0.0356mm 0.0356mm 0.0356mm 0.0356mm 0.0356mm 0.0356mm 0.0356mm 0.0356mm 0.0356mm 0.035559375mm"/>
+<param name="mtIsolate" value="1.6mm 0.1499mm 0.2007mm 0.1499mm 0.2007mm 0.1499mm 0.2007mm 0.1499mm 0.2007mm 0.1499mm 0.2007mm 0.1499mm 0.2007mm 0.1499mm 0.2007mm"/>
+<param name="mdWireWire" value="6mil"/>
+<param name="mdWirePad" value="6mil"/>
+<param name="mdWireVia" value="6mil"/>
+<param name="mdPadPad" value="6mil"/>
+<param name="mdPadVia" value="6mil"/>
+<param name="mdViaVia" value="6mil"/>
+<param name="mdSmdPad" value="6mil"/>
+<param name="mdSmdVia" value="6mil"/>
+<param name="mdSmdSmd" value="6mil"/>
+<param name="mdViaViaSameLayer" value="8mil"/>
 <param name="mnLayersViaInSmd" value="2"/>
-<param name="mdCopperDimension" value="40mil"/>
-<param name="mdDrill" value="15mil"/>
+<param name="mdCopperDimension" value="15mil"/>
+<param name="mdDrill" value="6mil"/>
 <param name="mdSmdStop" value="0mil"/>
-<param name="msWidth" value="12mil"/>
-<param name="msDrill" value="12mil"/>
-<param name="msMicroVia" value="9.99mm"/>
+<param name="msWidth" value="6mil"/>
+<param name="msDrill" value="10mil"/>
+<param name="msMicroVia" value="10mil"/>
 <param name="msBlindViaRatio" value="0.5"/>
 <param name="rvPadTop" value="0.25"/>
@@
 <param name="rvMicroViaOuter" value="0.25"/>
 <param name="rvMicroViaInner" value="0.25"/>
-<param name="rlMinPadTop" value="10mil"/>
+<param name="rlMinPadTop" value="5mil"/>
 <param name="rlMaxPadTop" value="20mil"/>
-<param name="rlMinPadInner" value="10mil"/>
+<param name="rlMinPadInner" value="5mil"/>
 <param name="rlMaxPadInner" value="20mil"/>
-<param name="rlMinPadBottom" value="10mil"/>
+<param name="rlMinPadBottom" value="5mil"/>
 <param name="rlMaxPadBottom" value="20mil"/>
-<param name="rlMinViaOuter" value="8mil"/>
+<param name="rlMinViaOuter" value="5mil"/>
 <param name="rlMaxViaOuter" value="20mil"/>
-<param name="rlMinViaInner" value="8mil"/>
+<param name="rlMinViaInner" value="5mil"/>
 <param name="rlMaxViaInner" value="20mil"/>
-<param name="rlMinMicroViaOuter" value="4mil"/>
+<param name="rlMinMicroViaOuter" value="5mil"/>
 <param name="rlMaxMicroViaOuter" value="20mil"/>
-<param name="rlMinMicroViaInner" value="4mil"/>
+<param name="rlMinMicroViaInner" value="5mil"/>
 <param name="rlMaxMicroViaInner" value="20mil"/>
 <param name="psTop" value="-1"/>
@@
 <param name="mvStopFrame" value="1"/>
 <param name="mvCreamFrame" value="0"/>
-<param name="mlMinStopFrame" value="4mil"/>
-<param name="mlMaxStopFrame" value="4mil"/>
+<param name="mlMinStopFrame" value="2.5mil"/>
+<param name="mlMaxStopFrame" value="2.5mil"/>
 <param name="mlMinCreamFrame" value="0mil"/>
 <param name="mlMaxCreamFrame" value="0mil"/>
@@
 </elements>
 <signals>
-<signal name="GND" class="1">
+<signal name="GND">
 <contactref element="GRAV" pad="2"/>
 <contactref element="BME" pad="3"/>
@@
 <contactref element="EXTRA_IO" pad="6"/>
 <contactref element="SD_R" pad="3"/>
-<polygon width="0.1524" layer="1" rank="0">
+<polygon width="0.1524" layer="1">
 <vertex x="105.41" y="3.81"/>
 <vertex x="-6.35" y="3.81"/>
@@
 <vertex x="105.41" y="82.423"/>
 </polygon>
-<via x="10.16" y="25.146" extent="1-16" drill="0.35"/>
-<via x="10.033" y="28.575" extent="1-16" drill="0.35"/>
-<via x="6.35" y="28.448" extent="1-16" drill="0.35"/>
-<via x="6.35" y="25.146" extent="1-16" drill="0.35"/>
+<via x="10.033" y="27.686" extent="1-16" drill="0.35"/>
+<via x="9.906" y="24.765" extent="1-16" drill="0.35"/>
+<via x="5.842" y="27.559" extent="1-16" drill="0.35"/>
+<via x="5.842" y="24.765" extent="1-16" drill="0.35"/>
 </signal>
 <signal name="CS">
@@
 <wire x1="13.28" y1="51.727" x2="13.28" y2="49.770575" width="0.3048" layer="1"/>
 <wire x1="80.01" y1="64.77" x2="78.359" y2="63.119" width="0.3048" layer="1"/>
-<wire x1="66.2432" y1="57.809775" x2="65.405" y2="56.971575" width="0.3048" layer="1"/>
-<wire x1="66.2432" y1="60.1472" x2="66.2432" y2="57.809775" width="0.3048" layer="1"/>
+<wire x1="67.1322" y1="57.555775" x2="65.405" y2="55.828575" width="0.3048" layer="1"/>
+<wire x1="67.1322" y1="61.0362" x2="67.1322" y2="57.555775" width="0.3048" layer="1"/>
 <wire x1="65.405" y1="46.355" x2="41.91" y2="22.86" width="0.3048" layer="1"/>
 <wire x1="78.359" y1="63.119" x2="69.215" y2="63.119" width="0.3048" layer="1"/>
-<wire x1="69.215" y1="63.119" x2="66.2432" y2="60.1472" width="0.3048" layer="1"/>
-<wire x1="65.405" y1="56.971575" x2="65.405" y2="46.355" width="0.3048" layer="1"/>
+<wire x1="69.215" y1="63.119" x2="67.1322" y2="61.0362" width="0.3048" layer="1"/>
+<wire x1="65.405" y1="55.828575" x2="65.405" y2="46.355" width="0.3048" layer="1"/>
 <wire x1="41.91" y1="22.86" x2="41.91" y2="21.463" width="0.3048" layer="16"/>
 <wire x1="41.91" y1="21.463" x2="41.656" y2="21.209" width="0.3048" layer="16"/>
@@
 <wire x1="78.74" y1="21.463" x2="86.36" y2="21.463" width="0.3048" layer="1"/>
 <wire x1="86.36" y1="21.463" x2="77.851" y2="29.972" width="0.3048" layer="1"/>
-<wire x1="87.7316" y1="48.9966" x2="90.043" y2="51.308" width="0.3048" layer="1"/>
-<wire x1="87.7316" y1="46.1678625" x2="87.7316" y2="48.9966" width="0.3048" layer="1"/>
-<wire x1="77.851" y1="36.2872625" x2="87.7316" y2="46.1678625" width="0.3048" layer="1"/>
+<wire x1="90.043" y1="47.2092625" x2="90.043" y2="51.308" width="0.3048" layer="1"/>
+<wire x1="77.851" y1="35.0172625" x2="90.043" y2="47.2092625" width="0.3048" layer="1"/>
 <wire x1="90.043" y1="51.308" x2="89.535" y2="51.816" width="0.3048" layer="1"/>
 <wire x1="89.535" y1="51.816" x2="86.36" y2="51.816" width="0.3048" layer="1"/>
-<wire x1="77.851" y1="29.972" x2="77.851" y2="36.2872625" width="0.3048" layer="1"/>
+<wire x1="77.851" y1="29.972" x2="77.851" y2="35.0172625" width="0.3048" layer="1"/>
 <wire x1="97.79" y1="58.42" x2="95.25" y2="58.42" width="0.3048" layer="1"/>
 <wire x1="55.88" y1="63.5" x2="55.88" y2="64.135" width="0.3048" layer="1"/>
@@
 <contactref element="GEIGER" pad="1"/>
 <contactref element="ARDUINO" pad="2"/>
-<wire x1="35.56" y1="63.5" x2="35.56" y2="60.833" width="0.3048" layer="1"/>
-<wire x1="35.56" y1="60.833" x2="59.69" y2="60.833" width="0.3048" layer="1"/>
-<wire x1="59.69" y1="60.833" x2="59.69" y2="58.42" width="0.3048" layer="1"/>
+<wire x1="59.69" y1="58.42" x2="59.69" y2="60.198" width="0.3048" layer="1"/>
+<wire x1="59.69" y1="60.198" x2="59.309" y2="60.579" width="0.3048" layer="1"/>
+<wire x1="35.56" y1="61.976" x2="35.56" y2="63.5" width="0.3048" layer="1"/>
+<wire x1="59.309" y1="60.579" x2="36.957" y2="60.579" width="0.3048" layer="1"/>
+<wire x1="36.957" y1="60.579" x2="35.56" y2="61.976" width="0.3048" layer="1"/>
 </signal>
 <signal name="DS">
