File: Spring 2023/Electrical/Eagle Files/strato_cats/ASCEND_SP_23.brd (EAGLE design)
At the start: 111.8 x 78.7 mm, 12 parts

Commit message: not sure what changed
Parts:
- added EXTRA_IO1: (no value), SparkFun-Connectors:1X06
- moved EXTRA_IO 3.05 mm to (14.5, 63.5)
Connections:
- new net D6: ARDUINO.6, EXTRA_IO1.1
- new net D7: ARDUINO.7, EXTRA_IO1.2
- net 3V: now also ARDUINO.3.3V
- net 5V: now also EXTRA_IO1.5
- net GND: now also EXTRA_IO1.6
- net SCL: now also EXTRA_IO1.3
- net SDA: now also EXTRA_IO1.4
Routing:
- net D6: track 0.00 -> 72.5 mm
- net D7: track 0.00 -> 65.2 mm
- net SDA: track 136.8 -> 160.8 mm, vias 0 -> 1
- net 3V: track 0.00 -> 12.7 mm
- net 5V: track 241.3 -> 253.9 mm
- net SCL: track 153.9 -> 164.7 mm
- net D4: track 49.8 -> 45.5 mm
- net D5: track 47.3 -> 45.1 mm
Other:
- board text added: "2 layer"
- board text added: "VER 1"
