File: Spring 2023/Electrical/Eagle Files/strato_cats/schematic.sch (EAGLE design)
At the start: 7 parts

Commit message: finished board
Parts:
- removed JP4: (no value), adafruit:PINHD-1X8BIG
- added BATT: (no value), SparkFun-Connectors:CONN_02
- added EXTRA_IO: (no value), SparkFun-Connectors:CONN_06SILK_FEMALE_PTH
- added GEIGER: (no value), SparkFun-Connectors:CONN_04PTH
- added SD_R: (no value), adafruit:PINHD-1X8BIG
- renumbered B1 to ARDUINO, J2 to GRAV, J4 to 9DOF_1, J9 to 9DOF_2, JP2 to BME, JP3 to GUVA
Connections:
- removed net !CS!_VIN: 9DOF_1.6, ARDUINO.7
- removed net +3V3: JP4.2
- removed net 5V*3: 9DOF_1.2, 9DOF_2.6, ARDUINO.5V, BME.1, GRAV.1, GUVA.1, JP4.1
- removed net AD0/SDO_VIN: 9DOF_1.5
- removed net AUX_CL_VIN: 9DOF_2.5
- removed net AUX_DA_VIN: 9DOF_2.4
- removed net CD: JP4.8
- removed net DI: ARDUINO.51/MOSI, JP4.6
- removed net DO: ARDUINO.50/MISO, JP4.5
- removed net FSYNC_VIN: 9DOF_2.3
- removed net INT_VIN: 9DOF_2.2
- removed net N$2: BME.2
- removed net SDA/SDI_VIN: 9DOF_1.3, ARDUINO.20(SDA), BME.6, GRAV.4
- removed net SDO/ADR: BME.5
- new net 3V: 9DOF_1.2
- new net 5V: ARDUINO.5V, BATT.1, BME.1, EXTRA_IO.5, GEIGER.3, GRAV.1, GUVA.1, SD_R.1
- new net D4: ARDUINO.4, EXTRA_IO.1
- new net D5: ARDUINO.5, EXTRA_IO.2
- new net DS: ARDUINO.3, GEIGER.2
- new net NS: ARDUINO.2, GEIGER.1
- new net SDA: 9DOF_1.3, ARDUINO.SDA, BME.6, EXTRA_IO.4, GRAV.4
- new net SDI: ARDUINO.51/MOSI, SD_R.6
- new net SDO: ARDUINO.50/MISO, SD_R.5
- net CLK: now also SD_R.4; no longer JP4.4
- net CS: now also SD_R.7; no longer BME.7, JP4.7
- net GND: now also ARDUINO.GND@2, ARDUINO.GND@3, BATT.2, EXTRA_IO.6, GEIGER.4, SD_R.3; no longer JP4.3
- net SCL: now also ARDUINO.SCL, EXTRA_IO.3; no longer ARDUINO.21(SCL)
Other:
- note removed: "SD"

Commit message: not sure what changed
Parts:
- added EXTRA_IO1: (no value), SparkFun-Connectors:CONN_06SILK_FEMALE_PTH
Connections:
- new net D6: ARDUINO.6, EXTRA_IO1.1
- new net D7: ARDUINO.7, EXTRA_IO1.2
- net 3V: now also ARDUINO.3.3V
- net 5V: now also EXTRA_IO1.5
- net GND: now also EXTRA_IO1.6
- net SCL: now also EXTRA_IO1.3
- net SDA: now also EXTRA_IO1.4
Changed lines of the file:
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@@
 <part name="EXTRA_IO" library="SparkFun-Connectors" deviceset="CONN_06" device="SILK_FEMALE_PTH"/>
 <part name="SD_R" library="adafruit" deviceset="PINHD-1X8" device="BIG"/>
+<part name="EXTRA_IO1" library="SparkFun-Connectors" deviceset="CONN_06" device="SILK_FEMALE_PTH"/>
 </parts>
 <sheets>
@@
 <attribute name="VALUE" x="-201.93" y="71.12" size="1.778" layer="96"/>
 </instance>
+<instance part="EXTRA_IO1" gate="G$1" x="-279.4" y="157.48" smashed="yes">
+<attribute name="VALUE" x="-284.48" y="147.574" size="1.778" layer="96" font="vector"/>
+<attribute name="NAME" x="-284.48" y="168.148" size="5.08" layer="95" font="vector"/>
+</instance>
 </instances>
 <busses>
@@
 <wire x1="-198.12" y1="88.9" x2="-210.82" y2="88.9" width="0.1524" layer="91"/>
 <label x="-210.82" y="88.9" size="1.778" layer="95"/>
+</segment>
+<segment>
+<pinref part="EXTRA_IO1" gate="G$1" pin="6"/>
+<wire x1="-274.32" y1="165.1" x2="-261.62" y2="165.1" width="0.1524" layer="91"/>
+<label x="-264.16" y="165.1" size="1.778" layer="95"/>
 </segment>
 </net>
@@
 <label x="-58.42" y="165.1" size="1.778" layer="95"/>
 </segment>
+<segment>
+<pinref part="EXTRA_IO1" gate="G$1" pin="3"/>
+<wire x1="-274.32" y1="157.48" x2="-261.62" y2="157.48" width="0.1524" layer="91"/>
+<label x="-264.16" y="157.48" size="1.778" layer="95"/>
+</segment>
 </net>
 <net name="SDO" class="0">
@@
 <label x="-58.42" y="162.56" size="1.778" layer="95"/>
 </segment>
+<segment>
+<pinref part="EXTRA_IO1" gate="G$1" pin="4"/>
+<wire x1="-274.32" y1="160.02" x2="-261.62" y2="160.02" width="0.1524" layer="91"/>
+<label x="-264.16" y="160.02" size="1.778" layer="95"/>
+</segment>
 </net>
 <net name="5V" class="0">
@@
 <wire x1="-198.12" y1="93.98" x2="-210.82" y2="93.98" width="0.1524" layer="91"/>
 <label x="-210.82" y="93.98" size="1.778" layer="95"/>
+</segment>
+<segment>
+<pinref part="EXTRA_IO1" gate="G$1" pin="5"/>
+<wire x1="-274.32" y1="162.56" x2="-261.62" y2="162.56" width="0.1524" layer="91"/>
+<label x="-264.16" y="162.56" size="1.778" layer="95"/>
 </segment>
 </net>
@@
 <label x="-58.42" y="160.02" size="1.778" layer="95"/>
 </segment>
-</net>
+<segment>
+<wire x1="-73.66" y1="81.28" x2="-68.58" y2="81.28" width="0.1524" layer="91"/>
+<pinref part="ARDUINO" gate="B1" pin="3.3V"/>
+<label x="-76.2" y="81.28" size="1.778" layer="95"/>
+</segment>
+</net>
+<net name="D6" class="0">
+<segment>
+<pinref part="ARDUINO" gate="B1" pin="6"/>
+<wire x1="-38.1" y1="53.34" x2="-30.48" y2="53.34" width="0.1524" layer="91"/>
+<label x="-30.48" y="53.34" size="1.778" layer="95"/>
+</segment>
+<segment>
+<pinref part="EXTRA_IO1" gate="G$1" pin="1"/>
+<wire x1="-274.32" y1="152.4" x2="-261.62" y2="152.4" width="0.1524" layer="91"/>
+<label x="-264.16" y="152.4" size="1.778" layer="95"/>
+</segment>
+</net>
+<net name="D7" class="0">
+<segment>
+<pinref part="ARDUINO" gate="B1" pin="7"/>
+<wire x1="-38.1" y1="55.88" x2="-30.48" y2="55.88" width="0.1524" layer="91"/>
+<label x="-30.48" y="55.88" size="1.778" layer="95"/>
+</segment>
+<segment>
+<pinref part="EXTRA_IO1" gate="G$1" pin="2"/>
+<wire x1="-274.32" y1="154.94" x2="-261.62" y2="154.94" width="0.1524" layer="91"/>
+<label x="-264.16" y="154.94" size="1.778" layer="95"/>
+</segment>
+</net>
